File: SmartBMS_2209A_Hardware/pasive_balance_rev4.kicad_sch (KiCad schematic)
At the start: 287 parts, among them IC1 BQ76PL455ATPFCTQ1, IC3 SI2319DS-T1-E3, IC5 2N7002E-T1-E3, IC6 ESP32-S3-WROOM-1-N8R2, J1 L-KLS1-218B-2-16-S-2X8X3, J10 Conn_01x02_Pin, J2 DE9_Plug_MountingHoles, J3 DS1022-06-2X3S81SR, J5 0015913124, J6 15-91-3044, J8 1757394, J9 10118194-0001LF, Q1 ZXTN4004KTC, Q10 7NM70G-TN3-R, Q11 7NM70G-TN3-R, Q12 7NM70G-TN3-R, Q13 7NM70G-TN3-R, Q14 7NM70G-TN3-R, Q15 7NM70G-TN3-R, Q16 7NM70G-TN3-R, Q17 7NM70G-TN3-R, Q18 TLP293_BL-TPL,E, Q19 TLP293_BL-TPL,E, Q2 7NM70G-TN3-R, Q20 UMH3N, Q21 7NM70G-TN3-R, Q22 7NM70G-TN3-R, Q23 7NM70G-TN3-R, Q24 7NM70G-TN3-R, Q25 7NM70G-TN3-R, Q26 7NM70G-TN3-R, Q27 7NM70G-TN3-R, Q28 7NM70G-TN3-R, Q29 7NM70G-TN3-R, Q3 7NM70G-TN3-R, Q30 7NM70G-TN3-R, Q31 7NM70G-TN3-R, Q32 7NM70G-TN3-R, Q33 7NM70G-TN3-R, Q34 7NM70G-TN3-R, Q35 7NM70G-TN3-R, Q36 7NM70G-TN3-R, Q4 7NM70G-TN3-R, Q5 7NM70G-TN3-R, Q6 7NM70G-TN3-R, Q7 7NM70G-TN3-R, Q8 7NM70G-TN3-R, Q9 7NM70G-TN3-R, U1 TJA1051T,118, U2 AMS1117-3.3, U3 CH340G, U4 BD9G341EFJ

Commit message: last 5.03.25
Parts:
- removed BAT0, BAT1, BAT10, BAT11, BAT12, BAT13, BAT14, BAT15, BAT16, BAT2, BAT3, BAT4, BAT5, BAT6, BAT7, BAT8, BAT9, CHP1, COMMH+1, COMMH-1, COMML+1, COMML-1, FAULTH+1, FAULTH-1, FAULTL+1, FAULTL-1, OUT1, V5VA0, VDIG1, VIO1, VM1, VP1, VREF1: 5002, Samacsys:5002, symbol dk_Test-Points:5002
- removed C1, C11, C2, C20, C3, C49, C51: GRM21BR71C475KA73L, Samacsys:CAPC2012X145N, symbol Kicad Plugin Symbol:GRM21BR71C475KA73L
- removed C10: GRM31CR72A105KA01L, Samacsys:CAPC3216X180N, symbol Kicad Plugin Symbol:GRM31CR72A105KA01L
- removed C12, C13, C15, C18, C19, C21, C22, C47, C8: C1608X7R1C104K, Samacsys:CAPC1608X90N, symbol Kicad Plugin Symbol:C1608X7R1C104K
- removed C14: GRM31CR71H475KA12L, Samacsys:CAPC3216X180N, symbol Kicad Plugin Symbol:GRM31CR71H475KA12L
- removed C16, C17, C24, C25, C28, C29, C32, C34, C55, C56, C57, C58, C59, C60, C61, C62: GRM32CR72A105KA35L, Samacsys:CAPC3225X180N, symbol Kicad Plugin Symbol:GRM32CR72A105KA35L
- removed C23: AEF1010330M100R, Samacsys:AEF1010330M100R, symbol Kicad Plugin Symbol:AEF1010330M100R
- removed C26, C30, C50, C52, C53, C6, C9: C0603X104K3RACTU, Samacsys:C0603, symbol Kicad Plugin Symbol:C0603X104K3RACTU
- removed C27: EEE-FH1C221L, SamacSys_Parts:EEETC1V470P, symbol SamacSys_Parts:EEE-FH1C221L
- removed C4: C0805C104K1RACTU, Samacsys:C0805, symbol Kicad Plugin Symbol:C0805C104K1RACTU
- removed C5: 08055A391JAT2A, Samacsys:CAPC2012X94N, symbol Kicad Plugin Symbol:08055A391JAT2A
- removed C54: C1608X7R1C105K080AC, Samacsys:CAPC1608X80N, symbol Kicad Plugin Symbol:C1608X7R1C105K080AC
- removed C7: C1210C185K3RACTU, Samacsys:C1210, symbol Kicad Plugin Symbol:C1210C185K3RACTU
- removed D1: 1N5819HW-7-F, digikey-footprints:SOD-123, symbol dk_Diodes-Rectifiers-Single:1N5819HW-7-F
- removed D10, D11, D12, D13, D14, D15, D16, D2: PESD5V0U1UA,115, Samacsys:SOD2512X110N, symbol Kicad Plugin Symbol:PESD5V0U1UA,115
- removed D17: SS54F-HF, Samacsys:SODFL4626X120N, symbol Kicad Plugin Symbol:SS54F-HF
- removed D18: SMCJ40CAQ-TP, SamacSys_Parts:DIOM7959X262N, symbol Samacsys:SMCJ40CAQ-TP
- removed D19: FSV20120V, Samacsys:FES10D, symbol Samacsys:FSV20120V
- removed D3: CDSOT23-SM712, digikey-footprints:SOT-23-3, symbol dk_TVS-Diodes:CDSOT23-SM712
- removed D4, D5, D7, D8: 1N4148W-7-F, digikey-footprints:SOD-123, symbol dk_Diodes-Rectifiers-Single:1N4148W-7-F
- removed D6: SMAJ90A, Diode_SMD:D_SMA, symbol Diode:SMAJ90A
- removed D9: 1N5819WS, Diode_SMD:D_SOD-323, symbol Diode:1N5819WS
- removed IC1: BQ76PL455ATPFCTQ1, Samacsys:QFP50P1400X1400X120-80N, symbol Kicad Plugin Symbol:BQ76PL455ATPFCTQ1
- removed IC3: SI2319DS-T1-E3, Samacsys:SOT95P237X112-3N, symbol Kicad Plugin Symbol:SI2319DS-T1-E3
- removed IC5: 2N7002E-T1-E3, Samacsys:SOT95P237X112-3N, symbol Kicad Plugin Symbol:2N7002E-T1-E3
- removed IC6: ESP32-S3-WROOM-1-N8R2, Samacsys:ESP32S3WROOM1N8R2, symbol Samacsys_kicad_sym:ESP32-S3-WROOM-1-N8R2
- removed J1: L-KLS1-218B-2-16-S-2X8X3, Connector_PinHeader_2.00mm:PinHeader_2x08_P2.00mm_Vertical, symbol Connector_Generic:Conn_02x08_Odd_Even
- removed J10: Conn_01x02_Pin, Connector_PinHeader_2.54mm:PinHeader_1x02_P2.54mm_Vertical, symbol Connector:Conn_01x02_Pin
- removed J2: DE9_Plug_MountingHoles, Connector_Dsub:DSUB-9_Female_Horizontal_P2.77x2.84mm_EdgePinOffset4.94mm_Housed_MountingHolesOffset7.48mm, symbol Connector:DE9_Plug_MountingHoles
- removed J3: DS1022-06-2X3S81SR, Connector_PinHeader_2.54mm:PinHeader_2x03_P2.54mm_Vertical, symbol Connector_Generic:Conn_02x03_Top_Bottom
- removed J5: 0015913124, Snapeda:0015913124, symbol Snapeda_Symbols:0015913244
- removed J6: 15-91-3044, Samacsys:15913044, symbol Kicad Plugin Symbol:15-91-3044
- removed J8: 1757394, Samacsys:1757394, symbol Samacsys:1757394
- removed J9: 10118194-0001LF, digikey-footprints:USB_Micro_B_Female_10118194-0001LF, symbol dk_USB-DVI-HDMI-Connectors:10118194-0001LF
- removed JP1: 120ohm EN, Jumper:SolderJumper-2_P1.3mm_Bridged2Bar_Pad1.0x1.5mm, symbol Jumper:SolderJumper_2_Bridged
- removed JP2: GND COM, Jumper:SolderJumper-2_P1.3mm_Bridged2Bar_Pad1.0x1.5mm, symbol Jumper:SolderJumper_2_Bridged
- removed L1: SRN4018BTA-330M, SamacSys_Parts:SRN4018BTA330M, symbol SamacSys_Parts:SRN4018BTA-330M
- removed L2: B82793C475N265, B82793C475N265, symbol SamacSys_Parts:B82793C475N265
- removed LED1, LED4: HSMH-C150, Samacsys:LEDC3216X120N, symbol Kicad Plugin Symbol:HSMH-C150
- removed LED2: 150060GS55040, Samacsys:LEDC1608X50N, symbol Kicad Plugin Symbol:150060GS55040
- removed LED3: HSMG-C150, Samacsys:LEDC3216X120N, symbol Kicad Plugin Symbol:HSMG-C150
- removed Q1: ZXTN4004KTC, Samacsys:ZXTN4004KTC, symbol Kicad Plugin Symbol:ZXTN4004KTC
- removed Q10, Q11, Q12, Q13, Q14, Q15, Q16, Q17, Q2, Q21, Q22, Q23, Q24, Q25, Q26, Q27, Q28, Q29, Q3, Q30, Q31, Q32, Q33, Q34, Q35, Q36, Q4, Q5, Q6, Q7, Q8, Q9: 7NM70G-TN3-R, Package_TO_SOT_SMD:TO-252-2, symbol Transistor_FET:QM6006D
- removed Q18, Q19: TLP293_BL-TPL,E, Samacsys:SOIC127P700X230-4N, symbol Kicad Plugin Symbol:TLP293_BL-TPL,E
- removed Q20: UMH3N, Package_TO_SOT_SMD:SOT-363_SC-70-6, symbol Transistor_BJT:UMH3N
- removed R1, R41, R42, R51, R53, R54, R6: CRCW060349R9FKEA, Samacsys:RESC1608X50N, symbol Kicad Plugin Symbol:CRCW060349R9FKEA
- removed R10, R13, R16, R19, R22, R25, R32, R33, R56, R59, R62, R65, R68, R7, R71, R74, R77, R80, R83, R84: CRCW06031K00FKEA, Samacsys:RESC1608X50N, symbol Kicad Plugin Symbol:CRCW06031K00FKEA
- removed R100, R3, R4, R86, R88, R90, R92, R95, R96, R99: CRCW060310R0FKEA, Samacsys:RESC1608X50N, symbol Kicad Plugin Symbol:CRCW060310R0FKEA
- removed R101, R12, R15, R18, R21, R24, R28, R29, R30, R37, R38, R39, R40, R52, R55, R58, R61, R64, R67, R70, R73, R76, R79, R82: RC0603FR-07100KL, Samacsys:RESC1608X55N, symbol Kicad Plugin Symbol:RC0603FR-07100KL
- removed R102: RC0603FR-0720KL, Samacsys:RESC1608X55N, symbol Kicad Plugin Symbol:RC0603FR-07100KL
- removed R103: 603-RC0603FR-0747KL, Samacsys:RESC1608X55N, symbol Kicad Plugin Symbol:RC0603FR-07100KL
- removed R104: RC0603FR-07750RL, Samacsys:RESC1608X55N, symbol Kicad Plugin Symbol:RC0603FR-07100KL
- removed R105: RC0603FR-073KL, Samacsys:RESC1608X55N, symbol Kicad Plugin Symbol:RC0603FR-07100KL
- removed R106, R107: RK73H1HRTTCM60R4F, Samacsys:RESC1608X50N, symbol Kicad Plugin Symbol:CRCW060349R9FKEA
- removed R11, R14, R17, R20, R23, R26, R31, R34, R36, R57, R60, R63, R66, R69, R72, R75, R78, R81, R9: CRCW06032K00FKEA, Samacsys:RESC1608X50N, symbol Kicad Plugin Symbol:CRCW06032K00FKEA
- removed R2: CRCW1206100RFKEA, Samacsys:RESC3216X60N, symbol Kicad Plugin Symbol:CRCW1206100RFKEA
- removed R27, R43, R44, R45, R46, R47, R48, R49, R50: CRCW120610R0FKEA, Samacsys:RESC3216X60N, symbol Kicad Plugin Symbol:CRCW120610R0FKEA
- removed R35, R85, R87, R89, R91, R93, R94, R97, R98: CRCW060310K0FKEA, Samacsys:RESC1608X50N, symbol Kicad Plugin Symbol:CRCW060310K0FKEA
- removed R5, R8: RC0603FR-071RL, Samacsys:RESC1608X55N, symbol Kicad Plugin Symbol:RC0603FR-071RL
- removed S1: GDH04S04, Samacsys:SOIC127P813X256-8N, symbol Kicad Plugin Symbol:GDH04S04
- removed S2, S3: SKQGADE010, SamacSys_Parts:SKQGAKE010, symbol SamacSys_Parts:SKQGADE010
- removed TP1: MAX VOLTAGE, TestPoint:TestPoint_Bridge_Pitch2.54mm_Drill1.3mm, symbol Connector:TestPoint
- removed TP6: GND, TestPoint:TestPoint_Bridge_Pitch2.54mm_Drill1.3mm, symbol Connector:TestPoint
- removed U1: TJA1051T,118, Package_SO:SOIC-8_3.9x4.9mm_P1.27mm, symbol Interface_CAN_LIN:TJA1051T
- removed U2: AMS1117-3.3, Package_TO_SOT_SMD:SOT-223-3_TabPin2, symbol Regulator_Linear:AMS1117-3.3
- removed U3: CH340G, Package_SO:SOIC-16_3.9x9.9mm_P1.27mm, symbol Interface_USB:CH340G
- removed U4: BD9G341EFJ, Package_SO:HTSOP-8-1EP_3.9x4.9mm_P1.27mm_EP2.4x3.2mm_ThermalVias, symbol Regulator_Switching:BD9G341EFJ
- removed Z1, Z10, Z11, Z12, Z13, Z14, Z15, Z16, Z2, Z3, Z4, Z5, Z6, Z7, Z8, Z9: DDZ6V2B-7, Samacsys:SOD3716X145N, symbol Kicad Plugin Symbol:DDZ6V2B-7
- added J8: DE9_Plug_MountingHoles, Connector_Dsub:DSUB-9_Female_Horizontal_P2.77x2.84mm_EdgePinOffset4.94mm_Housed_MountingHolesOffset7.48mm, symbol Library:DE9_Plug_MountingHoles
- added JP2: GND COM, Jumper:SolderJumper-2_P1.3mm_Bridged2Bar_Pad1.0x1.5mm, symbol Library:SolderJumper_2_Bridged
Connections:
- new net BQ76PL455/CELL0: JP2.1 (A)
- new net BQ76PL455/GND_COMM: JP2.2 (B)
- new net MCU/CANH: J8.7
- new net MCU/CANL: J8.2
- new net MCU/GND_: J8.0 (PAD)
- new net MCU/_GND: J8.3
- no-connect marks 7 -> 6
Other:
- added sheet BQ76PL455 (BQ76PL455.kicad_sch)
- added sheet BalanceMosfets (BalanceMosfets.kicad_sch)
- added sheet Connector (Connector.kicad_sch)
- added sheet DCDC_Converter (DCDC_Converter.kicad_sch)
- added sheet MCU (MCU.kicad_sch)
- note removed: "BQ76PL455ATPFCTQ1 & SOCK DIAGRAMS"
- note removed: "INTERFACES"
- note removed: "POWER DIAGRAMS"
- note removed: "TMS5701224CPGEQQ1 & SOCK DIAGRAMS"
- note removed: "cell0 to gnd1 is thick trace"
- company: OttomotiveTech -> (none)
- title: ott_bmu -> SmartBMS2209A
